Commit message: add discontinuous gait

File: spotmicro/spotmicro/urdf/spotmicro.xacro (robot description, xacro)
@@ -51,5 +51,5 @@
         <material>Gazebo/Black</material>
         <kp>1000000.0</kp>
-        <kd>1000.0</kd>
+        <kd>100.0</kd>
         <mu1>100</mu1>
         <mu2>100</mu2>
@@ -90,5 +90,5 @@
         <material>Gazebo/Yellow</material>
         <kp>1000000.0</kp>
-        <kd>1000.0</kd>
+        <kd>100.0</kd>
         <mu1>100</mu1>
         <mu2>100</mu2>
@@ -129,5 +129,5 @@
         <material>Gazebo/Black</material>
         <kp>1000000.0</kp>
-        <kd>1000.0</kd>
+        <kd>100.0</kd>
         <mu1>100</mu1>
         <mu2>100</mu2>
@@ -157,6 +157,6 @@
         <material>Gazebo/Black</material>
         <kp>1000000.0</kp>
-        <kd>1000.0</kd>
-        <mu1>100</mu1>
+        <kd>1.0</kd>
+        <mu1>200</mu1>
         <mu2>100</mu2>
     </gazebo>
@@ -194,10 +194,12 @@
         <origin rpy="0 0 0" xyz="0 0 0"/>
     </collision>
-    <xacro:box_inertial x="0.24" y="0.11" z="0.065" mass="1.0"/>
+    <xacro:box_inertial_with_origin x="0.24" y="0.11" z="0.065" mass="0.6">
+        <origin xyz="0.05 0 0" rpy="0 0 0"/>
+    </xacro:box_inertial_with_origin>
 </link>
 <gazebo reference="base_link">
         <material>Gazebo/Yellow</material>
         <kp>1000000.0</kp>
-        <kd>1000.0</kd>
+        <kd>100.0</kd>
         <mu1>100</mu1>
         <mu2>100</mu2>
