Commit message: add weight_shift configurable param for walk_gait and discontinuous_gait

File: spotmicro/urdf/spotmicro.xacro (robot description, xacro)
@@ -195,5 +195,5 @@
     </collision>
     <xacro:box_inertial_with_origin x="0.24" y="0.11" z="0.065" mass="0.6">
-        <origin xyz="0.05 0 0" rpy="0 0 0"/>
+        <origin xyz="0.0 0 0" rpy="0 0 0"/>
     </xacro:box_inertial_with_origin>
 </link>

Commit message: puppy branch

File: spotmicro/urdf/spotmicro.xacro (robot description, xacro)
@@ -2,12 +2,12 @@
 <robot name="spotmicro" xmlns:xacro="http://ros.org/wiki/xacro">
 <xacro:property name="radius" value="0.01" />
-<xacro:property name="offset_y" value="0.04" />
-<xacro:property name="offset_x" value="0.09" />
-<xacro:property name="offset_z" value="0.01" />
-<xacro:property name="a" value="0.01" />
-<xacro:property name="b" value="0.055" />
-<xacro:property name="c" value="0.11" />
-<xacro:property name="d" value="0.01" />
-<xacro:property name="e" value="0.115" />
+<xacro:property name="offset_y" value="0.0265" />
+<xacro:property name="offset_x" value="0.055" />
+<xacro:property name="offset_z" value="0.0" />
+<xacro:property name="a" value="0.006" />
+<xacro:property name="b" value="0.02" />
+<xacro:property name="c" value="0.055" />
+<xacro:property name="d" value="0.005" />
+<xacro:property name="e" value="0.055" />
 <xacro:include filename="$(find spotmicro)/urdf/common.xacro" />
 <material name="black">
@@ -17,26 +17,36 @@
     <color rgba="1.0 1.0 0.0 1.0"/>
   </material>
+    <material name="white">
+    <color rgba="1 1 1 1.0"/>
+  </material>
 <xacro:macro name="leg" params="name l f">
-	<joint name="${name}0" type="revolute">
+    <joint name="${name}0" type="revolute">
         <parent link="base_link"/>
         <child link="${name}a"/>
         <axis xyz="1 0 0"/>
         <origin xyz="${offset_x*f} ${offset_y*l} ${offset_z}" rpy="0 0 0"/>
-        <limit lower="${-pi/4}" upper="${pi/4}" effort="1000.0" velocity="1.5"/>
+        <limit lower="${-pi/4}" upper="${pi/4}" effort="1000.0" velocity="2"/>
     </joint>
     <link name="${name}a">
-    	<visual>
-    		<geometry>
-                <box size="0.045 0.025 0.055" />
-    		</geometry>
-    		<origin xyz="0 0 ${-a}" rpy="0 0 0"/>
-            <material name="black"/>
-    	</visual>
-        <visual>
-            <geometry>
-                <cylinder radius="0.017" length="0.02"/>
-            </geometry>
-            <origin xyz="0 ${l*(0.025+0.02)/2} ${-a}" rpy="${pi/2} 0 0"/>
-            <material name="black"/>
+        <visual>
+            <geometry>
+                <box size="0.04 0.01 0.03" />
+            </geometry>
+            <origin xyz="0 0 0" rpy="0 0 0"/>
+            <material name="white"/>
+        </visual>
+        <visual>
+            <geometry>
+                <cylinder radius="0.005" length="0.008"/>
+            </geometry>
+            <origin xyz="${-0.005*f} ${l*0.009} ${a}" rpy="${pi/2} 0 0"/>
+            <material name="white"/>
+        </visual>
+        <visual>
+            <geometry>
+                <cylinder radius="0.005" length="0.008"/>
+            </geometry>
+            <origin xyz="${-0.005*f} ${l*0.009} ${-a}" rpy="${pi/2} 0 0"/>
+            <material name="white"/>
         </visual>
         <collision>
@@ -49,5 +59,5 @@
     </link>
     <gazebo reference="${name}a">
-        <material>Gazebo/Black</material>
+        <material>Gazebo/White</material>
         <kp>1000000.0</kp>
         <kd>100.0</kd>
@@ -59,34 +69,27 @@
         <child link="${name}b"/>
         <axis xyz="1 0 0"/>
-        <origin xyz="0 ${l*b} ${-a}" rpy="${-pi/2} 0 ${pi/2}"/>
-        <limit lower="${-pi/4}" upper="${pi*3/4}" effort="1000.0" velocity="1.5"/>
+        <origin xyz="${-0.005*f} ${l*b} ${-a}" rpy="${-pi/2} 0 ${pi/2}"/>
+        <limit lower="${-pi/4}" upper="${pi*3/4}" effort="1000.0" velocity="2"/>
     </joint>
     <link name="${name}b">
-    	<visual>
-    		<geometry>
-    			<box size="0.045 0.13 0.03"/>
-    		</geometry>
-    		<origin xyz="0 0.045 0" rpy="0 0 0"/>
-            <material name="yellow"/>
-    	</visual>
-        <visual>
-            <geometry>
-                <cylinder radius="0.017" length="0.055"/>
-            </geometry>
-            <origin xyz="0 ${c} ${-d}" rpy="0 ${pi/2} 0"/>
-            <material name="yellow"/>
-        </visual>
-        <collision>
-            <geometry>
-                <box size="0.045 0.13 0.03"/>
-            </geometry>
-            <origin xyz="0 0.045 0" rpy="0 0 0"/>
-        </collision>
-        <xacro:box_inertial_with_origin x="0.045" y="0.13" z="0.03" mass="0.07">
-            <origin xyz="0 0.045 0" rpy="0 0 0"/>
+        <visual>
+            <geometry>
+                <box size="0.005 ${c} 0.01"/>
+            </geometry>
+            <origin xyz="0 ${c/2} 0" rpy="0 0 0"/>
+            <material name="white"/>
+        </visual>
+        <collision>
+            <geometry>
+                <box size="0.005 ${c} 0.01"/>
+            </geometry>
+            <origin xyz="0 ${c/2} 0" rpy="0 0 0"/>
+        </collision>
+        <xacro:box_inertial_with_origin x="0.005" y="${c}" z="0.01" mass="0.01">
+            <origin xyz="0 ${c/2} 0" rpy="0 0 0"/>
         </xacro:box_inertial_with_origin>
     </link>
     <gazebo reference="${name}b">
-        <material>Gazebo/Yellow</material>
+        <material>Gazebo/White</material>
         <kp>1000000.0</kp>
         <kd>100.0</kd>
@@ -98,34 +101,27 @@
         <child link="${name}c"/>
         <axis xyz="1 0 0"/>
-        <origin xyz="0 ${c} ${-d}" rpy="${-pi} 0 0"/>
-        <limit lower="${pi/4}" upper="${pi}" effort="1000.0" velocity="1.5"/>
+        <origin xyz="${-d*l} ${c} 0" rpy="${-pi} 0 0"/>
+        <limit lower="0" upper="${pi}" effort="1000.0" velocity="2"/>
     </joint>
     <link name="${name}c">
         <visual>
             <geometry>
-                <box size="0.045 0.045 0.025"/>
-            </geometry>
-            <origin xyz="0 0.01 0" rpy="0 0 0"/>
-            <material name="black"/>
-        </visual>
-    	<visual>
-    		<geometry>
-    			<box size="0.02 0.115 0.02"/>
-    		</geometry>
-    		<origin xyz="0 0.055 0" rpy="0 0 0"/>
-            <material name="black"/>
-    	</visual>
-        <collision>
-            <geometry>
-                <box size="0.045 0.115 0.025"/>
-            </geometry>
-            <origin xyz="0 0.045 0" rpy="0 0 0"/>
-        </collision>
-        <xacro:box_inertial_with_origin x="0.045" y="0.045" z="0.025" mass="0.06">
-            <origin xyz="0 0.01 0" rpy="0 0 0"/>
+                <box size="${d} ${e+0.025} 0.01"/>
+            </geometry>
+            <origin xyz="0 ${(e-0.025)/2} 0" rpy="0 0 0"/>
+            <material name="white"/>
+        </visual>
+        <collision>
+            <geometry>
+                <box size="${d} ${e+0.025} 0.01"/>
+            </geometry>
+            <origin xyz="0 ${(e-0.025)/2} 0" rpy="0 0 0"/>
+        </collision>
+        <xacro:box_inertial_with_origin x="${d}" y="${e+0.025}" z="0.01" mass="0.01">
+            <origin xyz="0 ${(e-0.025)/2} 0" rpy="0 0 0"/>
         </xacro:box_inertial_with_origin>
     </link>
     <gazebo reference="${name}c">
-        <material>Gazebo/Black</material>
+        <material>Gazebo/White</material>
         <kp>1000000.0</kp>
         <kd>100.0</kd>
@@ -133,5 +129,5 @@
         <mu2>100</mu2>
     </gazebo>
-    <joint name="${name}3" type="fixed">
+    <joint name="${name}t" type="fixed">
         <parent link="${name}c"/>
         <child link="${name}d"/>
@@ -141,19 +137,83 @@
         <visual>
             <geometry>
-                <sphere radius="0.02"/>
+                <sphere radius="0.01"/>
             </geometry>
             <origin xyz="0 0 0" rpy="0 0 0"/>
-            <material name="black"/>
-        </visual>
-        <collision>
-            <geometry>
-                <sphere radius="0.02"/>
+            <material name="white"/>
+        </visual>
+        <collision>
+            <geometry>
+                <sphere radius="0.01"/>
             </geometry>
             <origin xyz="0 0 0" rpy="0 0 0"/>
         </collision>
-        <xacro:sphere_inertial radius="0.02" mass="0.01"/>
+        <xacro:sphere_inertial radius="0.01" mass="0.001"/>
     </link>
     <gazebo reference="${name}d">
-        <material>Gazebo/Black</material>
+        <material>Gazebo/White</material>
+        <kp>1000000.0</kp>
+        <kd>1.0</kd>
+        <mu1>200</mu1>
+        <mu2>100</mu2>
+    </gazebo>
+    <joint name="${name}3" type="revolute">
+        <parent link="${name}a"/>
+        <child link="${name}e"/>
+        <axis xyz="1 0 0"/>
+        <origin xyz="${-0.005*f} ${l*b} ${a}" rpy="0 0 ${pi/2}"/>
+        <limit lower="${-pi/4}" upper="${pi*3/4}" effort="1000.0" velocity="2"/>
+    </joint>
+    <link name="${name}e">
+        <visual>
+            <geometry>
+                <box size="0.005 0.024 0.01"/>
+            </geometry>
+            <origin xyz="0 ${0.024/2} 0" rpy="0 0 0"/>
+            <material name="white"/>
+        </visual>
+        <collision>
+            <geometry>
+                <box size="0.005 0.024 0.01"/>
+            </geometry>
+            <origin xyz="0 ${0.024/2} 0" rpy="0 0 0"/>
+        </collision>
+        <xacro:box_inertial_with_origin x="0.005" y="0.024" z="0.01" mass="0.001">
+            <origin xyz="0 ${0.024/2} 0" rpy="0 0 0"/>
+        </xacro:box_inertial_with_origin>
+    </link>
+    <gazebo reference="${name}e">
+        <material>Gazebo/White</material>
+        <kp>1000000.0</kp>
+        <kd>1.0</kd>
+        <mu1>200</mu1>
+        <mu2>100</mu2>
+    </gazebo>
+    <joint name="${name}4" type="revolute">
+        <parent link="${name}e"/>
+        <child link="${name}f"/>
+        <axis xyz="1 0 0"/>
+        <origin xyz="${0.005*l} 0.024 0" rpy="${-pi} 0 0"/>
+        <limit lower="${-pi}" upper="${pi}" effort="1000.0" velocity="2"/>
+    </joint>
+    <link name="${name}f">
+        <visual>
+            <geometry>
+                <box size="0.005 0.055 0.005"/>
+            </geometry>
+            <origin xyz="0 ${0.055/2} 0" rpy="0 0 0"/>
+            <material name="white"/>
+        </visual>
+        <collision>
+            <geometry>
+                <box size="0.005 0.055 0.005"/>
+            </geometry>
+            <origin xyz="0 ${0.055/2} 0" rpy="0 0 0"/>
+        </collision>
+        <xacro:box_inertial_with_origin x="0.005" y="0.055" z="0.005" mass="0.005">
+            <origin xyz="0 ${0.055/2} 0" rpy="0 0 0"/>
+        </xacro:box_inertial_with_origin>
+    </link>
+    <gazebo reference="${name}f">
+        <material>Gazebo/White</material>
         <kp>1000000.0</kp>
         <kd>1.0</kd>
@@ -165,39 +225,40 @@
     <visual>
         <geometry>
-            <box size="0.24 0.05 0.065"/>
-        </geometry>
-        <material name="yellow"/>
+            <box size="0.16 0.02 0.02"/>
+        </geometry>
+        <material name="white"/>
     </visual>
     <visual>
         <geometry>
-            <box size="0.13 0.11 0.065"/>
-        </geometry>
-        <material name="yellow"/>
+            <box size="0.064 0.075 0.04"/>
+        </geometry>
+        <material name="white"/>
     </visual>
     <visual>
         <geometry>
-            <box size="0.05 0.11 0.065"/>
-        </geometry>
-        <origin xyz="${0.13/2+0.07} 0 0" rpy="0 0 0"/>
-        <material name="yellow"/>
+            <box size="0.003 0.075 0.04"/>
+        </geometry>
+        <origin xyz="${0.16/2-0.0015} 0 0" rpy="0 0 0"/>
+        <material name="white"/>
     </visual>
     <visual>
         <geometry>
-            <box size="0.05 0.11 0.065"/>
-        </geometry>
-        <origin xyz="${-0.13/2-0.07} 0 0" rpy="0 0 0"/>
+            <box size="0.003 0.075 0.04"/>
+        </geometry>
+        <origin xyz="${-0.16/2+0.0015} 0 0" rpy="0 0 0"/>
+        <material name="white"/>
     </visual>
     <collision>
         <geometry>
-            <box size="0.24 0.11 0.065"/>
+            <box size="0.16 0.075 0.04"/>
         </geometry>
         <origin rpy="0 0 0" xyz="0 0 0"/>
     </collision>
-    <xacro:box_inertial_with_origin x="0.24" y="0.11" z="0.065" mass="0.6">
+    <xacro:box_inertial_with_origin x="0.16" y="0.075" z="0.04" mass="0.3">
         <origin xyz="0.0 0 0" rpy="0 0 0"/>
     </xacro:box_inertial_with_origin>
 </link>
 <gazebo reference="base_link">
-        <material>Gazebo/Yellow</material>
+        <material>Gazebo/White</material>
         <kp>1000000.0</kp>
         <kd>100.0</kd>

Commit message: bug: gazebo sim

File: spotmicro/urdf/spotmicro.xacro (robot description, xacro)
@@ -13,11 +13,11 @@
 <material name="black">
     <color rgba="0.0 0.0 0.0 1.0"/>
-  </material>
-  <material name="yellow">
+</material>
+<material name="yellow">
     <color rgba="1.0 1.0 0.0 1.0"/>
-  </material>
-    <material name="white">
-    <color rgba="1 1 1 1.0"/>
-  </material>
+</material>
+<material name="white">
+    <color rgba="1.0 1.0 1.0 1.0"/>
+</material>
 <xacro:macro name="leg" params="name l f">
     <joint name="${name}0" type="revolute">
@@ -26,5 +26,5 @@
         <axis xyz="1 0 0"/>
         <origin xyz="${offset_x*f} ${offset_y*l} ${offset_z}" rpy="0 0 0"/>
-        <limit lower="${-pi/4}" upper="${pi/4}" effort="1000.0" velocity="2"/>
+        <limit lower="${-pi/4}" upper="${pi/4}" effort="1000.0" velocity="10.0"/>
     </joint>
     <link name="${name}a">
@@ -56,5 +56,5 @@
             <origin rpy="0 0 0" xyz="0 0 0"/>
         </collision>
-        <xacro:box_inertial x="0.24" y="0.11" z="0.065" mass="0.06"/>
+        <xacro:box_inertial x="0.24" y="0.11" z="0.065" mass="0.02"/>
     </link>
     <gazebo reference="${name}a">
@@ -70,5 +70,5 @@
         <axis xyz="1 0 0"/>
         <origin xyz="${-0.005*f} ${l*b} ${-a}" rpy="${-pi/2} 0 ${pi/2}"/>
-        <limit lower="${-pi/4}" upper="${pi*3/4}" effort="1000.0" velocity="2"/>
+        <limit lower="${-pi/4}" upper="${pi*3/4}" effort="1000.0" velocity="10.0"/>
     </joint>
     <link name="${name}b">
@@ -102,5 +102,5 @@
         <axis xyz="1 0 0"/>
         <origin xyz="${-d*l} ${c} 0" rpy="${-pi} 0 0"/>
-        <limit lower="0" upper="${pi}" effort="1000.0" velocity="2"/>
+        <limit lower="0" upper="${pi}" effort="1000.0" velocity="10.0"/>
     </joint>
     <link name="${name}c">
@@ -156,5 +156,5 @@
         <mu1>200</mu1>
         <mu2>100</mu2>
-    </gazebo>
+    </gazebo> -->
     <joint name="${name}3" type="revolute">
         <parent link="${name}a"/>
@@ -162,5 +162,5 @@
         <axis xyz="1 0 0"/>
         <origin xyz="${-0.005*f} ${l*b} ${a}" rpy="0 0 ${pi/2}"/>
-        <limit lower="${-pi/4}" upper="${pi*3/4}" effort="1000.0" velocity="2"/>
+        <limit lower="${-pi/4}" upper="${pi*3/4}" effort="1000.0" velocity="10.0"/>
     </joint>
     <link name="${name}e">
@@ -194,5 +194,5 @@
         <axis xyz="1 0 0"/>
         <origin xyz="${0.005*l} 0.024 0" rpy="${-pi} 0 0"/>
-        <limit lower="${-pi}" upper="${pi}" effort="1000.0" velocity="2"/>
+        <limit lower="${-pi}" upper="${pi}" effort="1000.0" velocity="10.0"/>
     </joint>
     <link name="${name}f">
@@ -286,18 +286,25 @@
    <xacro:transmission_block joint_name="lf1"/>
    <xacro:transmission_block joint_name="lf2"/>
+   <xacro:transmission_block joint_name="lf3"/>
+   <xacro:transmission_block joint_name="lf4"/>
    <xacro:transmission_block joint_name="rf0"/>
    <xacro:transmission_block joint_name="rf1"/>
    <xacro:transmission_block joint_name="rf2"/>
+   <xacro:transmission_block joint_name="rf3"/>
+   <xacro:transmission_block joint_name="rf4"/>
    <xacro:transmission_block joint_name="lr0"/>
    <xacro:transmission_block joint_name="lr1"/>
    <xacro:transmission_block joint_name="lr2"/>
+   <xacro:transmission_block joint_name="lr3"/>
+   <xacro:transmission_block joint_name="lr4"/>
    <xacro:transmission_block joint_name="rr0"/>
    <xacro:transmission_block joint_name="rr1"/>
    <xacro:transmission_block joint_name="rr2"/>
+   <xacro:transmission_block joint_name="rr3"/>
+   <xacro:transmission_block joint_name="rr4"/>
 <!-- ros_control plugin -->
   <gazebo>
     <plugin name="gazebo_ros_control" filename="libgazebo_ros_control.so">
       <!--<robotNamespace>/spotmicro</robotNamespace>-->
-      <robotSimType>motion_control/GaitHWSim</robotSimType>
     </plugin>
   </gazebo>

Commit message: readme

File: spotmicro/urdf/spotmicro.xacro (robot description, xacro)
@@ -156,5 +156,5 @@
         <mu1>200</mu1>
         <mu2>100</mu2>
-    </gazebo> -->
+    </gazebo>
     <joint name="${name}3" type="revolute">
         <parent link="${name}a"/>
@@ -270,5 +270,5 @@
 <xacro:leg name="rf" l="-1" f="1"/>
 <xacro:leg name="rr" l="-1" f="-1"/>
-<xacro:macro name="transmission_block" params="joint_name">
+    <xacro:macro name="transmission_block" params="joint_name">
       <transmission name="${joint_name}_tran">
         <type>transmission_interface/SimpleTransmission</type>
@@ -281,5 +281,5 @@
         </actuator>
       </transmission>
-   </xacro:macro>
+    </xacro:macro>
  <!-- Transmissions for ROS Control -->
    <xacro:transmission_block joint_name="lf0"/>
